Commit message: Add files via upload

File: description/example_gazebo.xacro (robot description, xacro)
@@ -45,4 +45,5 @@
                 <param name="max">3.14</param>
             </command_interface>
+            <command_interface name="velocity"/>
             <state_interface name="position">
                 <param name="initial_value">0.0</param>
@@ -52,4 +53,5 @@
         </joint>
         <joint name="joint_2">
+            <command_interface name="velocity"/>
             <command_interface name="position">
                 <param name="min">-3.14</param>
@@ -63,4 +65,5 @@
         </joint>
         <joint name="joint_3">
+            <command_interface name="velocity"/>
             <command_interface name="position">
                 <param name="min">-3.14</param>
@@ -80,20 +83,20 @@
         </plugin>
     </gazebo>
-    <gazebo reference="link0">
+    <gazebo reference="link_0">
         <mu1>0.2</mu1>
         <mu2>0.2</mu2>
         <material>Gazebo/Green</material>
     </gazebo>
-    <gazebo reference="link1">
+    <gazebo reference="link_1">
         <mu1>0.2</mu1>
         <mu2>0.2</mu2>
         <material>Gazebo/Green</material>
     </gazebo>
-    <gazebo reference="link2">
+    <gazebo reference="link_2">
         <mu1>0.2</mu1>
         <mu2>0.2</mu2>
         <material>Gazebo/Black</material>
     </gazebo>
-    <gazebo reference="link3">
+    <gazebo reference="link_3">
         <mu1>0.2</mu1>
         <mu2>0.2</mu2>

File: description/example_robot.urdf.xacro (robot description, xacro)
@@ -83,5 +83,5 @@
         <axis xyz="0 0 1"/>
         <limit lower="-3.14" upper="3.14" effort="1000" velocity="0.5"/>
-        <dynamics damping="0" friction="0"/>
+        <dynamics damping="0.1" friction="0.1"/>
     </joint>
     <link name="link_2">
@@ -117,5 +117,5 @@
         <axis xyz="0 0 1"/>
         <limit lower="-3.14" upper="3.14" effort="0.5" velocity="0.5"/>
-        <dynamics damping="10" friction="10"/>
+        <dynamics damping="0.1" friction="0.1"/>
     </joint>
     <link name="link_3">
@@ -148,5 +148,5 @@
         <axis xyz="0 0 1"/>
         <limit lower="-3.14" upper="3.14" effort="1000" velocity="0.5"/>
-        <dynamics damping="10" friction="10"/>
+        <dynamics damping="0.1" friction="0.1"/>
     </joint>
     <joint name="joint_eff" type="fixed">
